File: layout/led2ch_v0.2.brd (EAGLE design)
At the start: 34.8 x 28.3 mm, 28 parts, among them IC1 MCP16311T-E/MNY, U1 ESP-WROOM-32

Commit message: minor changes
Parts:
- L2: value XAL4040-153MEB 15uH -> XAL4040-153MEB / ASPI-4030S-150M-T 15uH
Changed lines of the file:
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@@
 <element name="U1" library="esp32" package="ESP-WROOM-32" value="ESP-WROOM-32" x="19.4" y="18.7" rot="R90"/>
 <element name="U$3" library="falkor" package="3X2-2.00RM" value="3X2-2.00RM" x="24.7" y="4.3" rot="R90"/>
-<element name="L2" library="Seeed-OPL-Inductor" package="L0420" value="XAL4040-153MEB 15uH" x="13.5" y="4.275" rot="R90">
+<element name="L2" library="Seeed-OPL-Inductor" package="L0420" value="XAL4040-153MEB / ASPI-4030S-150M-T 15uH" x="13.5" y="4.275" rot="R90">
 <attribute name="MPN" value="SPD3D16-4R7M" x="13.5" y="4.275" size="1.778" layer="27" font="vector" rot="R90" display="off"/>
 </element>
