File: layout/led2ch_v0.2.sch (EAGLE design)
At the start: 28 parts, among them IC1 MCP16311T-E/MNY, U1 ESP-WROOM-32

Commit message: minor changes
Parts:
- L2: value XAL4040-153MEB 15uH -> XAL4040-153MEB / ASPI-4030S-150M-T 15uH
Changed lines of the file:
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@@
 <part name="P+2" library="supply1" deviceset="+24V" device=""/>
 <part name="U$3" library="falkor" deviceset="3X2-2.00RM" device=""/>
-<part name="L2" library="Seeed-OPL-Inductor" deviceset="SMD-POWER-INDUCTOR-4.7UH-20%-750MA(2P-3.9X3.9MM)" device="" value="XAL4040-153MEB 15uH"/>
+<part name="L2" library="Seeed-OPL-Inductor" deviceset="SMD-POWER-INDUCTOR-4.7UH-20%-750MA(2P-3.9X3.9MM)" device="" value="XAL4040-153MEB / ASPI-4030S-150M-T 15uH"/>
 <part name="TP5" library="testpad" deviceset="TP" device="B1,27"/>
 <part name="TP6" library="testpad" deviceset="TP" device="B1,27"/>
